File: kicad/unibatch-9x9.kicad_pcb (KiCad board)
At the start: 2 copper layers, 50 x 50 mm, 113 parts, among them Q1 2N7002, Q2 2N7002, Q3 2N7002, Q4 2N7002, Q5 2N7002, Q6 2N7002, Q7 2N7002, Q8 2N7002, Q9 2N7002, SW1 SW_DPDT_x2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

Commit message: fixed some minor bugs
Routing:
- net VS: track 58.9 -> 62.9 mm, vias 1 -> 2
