File: kicad/unibatch-9x9.sch (KiCad schematic (older format))
At the start: 108 parts, among them Q1 2N7002, Q2 2N7002, Q3 2N7002, Q4 2N7002, Q5 2N7002, Q6 2N7002, Q7 2N7002, Q8 2N7002, Q9 2N7002, SW1 SW_DPDT_x2, U1 NE555D, U2 4017

Commit message: finished layout
Parts:
- BT1: footprint Battery:BatteryHolder_Keystone_1060_1x2032 -> Connector_PinHeader_2.54mm:PinHeader_1x02_P2.54mm_Vertical
- D1, D10, D11, D12, D13, D14, D15, D16, D17, D18, D19, D2, D20, D21, D22, D23, D24, D25, D26, D27, D28, D29, D3, D30, D31, D32, D33, D34, D35, D36, D37, D38, D39, D4, D40, D41, D42, D43, D44, D45, D46, D47, D48, D49, D5, D50, D51, D52, D53, D54, D55, D56, D57, D58, D59, D6, D60, D61, D62, D63, D64, D65, D66, D67, D68, D69, D7, D70, D71, D72, D73, D74, D75, D76, D77, D78, D79, D8, D80, D81, D9: footprint nibble++:LED_0805_2012Metric_Pad1.15x1.40mm_HandSolder_simple_drawing -> LED_SMD:LED_0805_2012Metric_Pad1.15x1.40mm_HandSolder
- R10, R11, R3, R4, R5, R6, R7, R8, R9: footprint (none) -> Resistor_SMD:R_0805_2012Metric_Pad1.15x1.40mm_HandSolder
- SW1: footprint nibble++:smd_switch_slide -> unibatch:smd_switch_slide
- U2: footprint nibble++:SOP-16_4.4x10.4mm_P1.27mm_simple_drawing -> unibatch:SOP-16_4.4x10.4mm_P1.27mm_simple_drawing
Other:
- note removed: "Vorwiderstand nötig?"

Commit message: fixed some minor bugs
Parts:
- BT1: value CR2023 -> Battery-Holder (2x AAA)
Other:
- moved on the sheet: BT1
Changed lines of the file:
@@
 L Device:Battery_Cell BT1
 U 1 1 5BE72A56
-P 650 900
-F 0 "BT1" H 768 996 50  0000 L CNN
-F 1 "CR2023" H 768 905 50  0000 L CNN
-F 2 "Connector_PinHeader_2.54mm:PinHeader_1x02_P2.54mm_Vertical" V 650 960 50  0001 C CNN
-F 3 "~" V 650 960 50  0001 C CNN
-	1    650  900
+P 650 1050
+F 0 "BT1" H 768 1146 50  0000 L CNN
+F 1 "Battery-Holder (2x AAA)" H 768 1055 50  0000 L CNN
+F 2 "Connector_PinHeader_2.54mm:PinHeader_1x02_P2.54mm_Vertical" V 650 1110 50  0001 C CNN
+F 3 "~" V 650 1110 50  0001 C CNN
+	1    650  1050
 	1    0    0    -1
 $EndComp
@@
 L power:GND #PWR05
 U 1 1 5BE72B54
-P 650 1000
-F 0 "#PWR05" H 650 750 50  0001 C CNN
-F 1 "GND" H 655 827 50  0000 C CNN
-F 2 "" H 650 1000 50  0001 C CNN
-F 3 "" H 650 1000 50  0001 C CNN
-	1    650  1000
+P 650 1150
+F 0 "#PWR05" H 650 900 50  0001 C CNN
+F 1 "GND" H 655 977 50  0000 C CNN
+F 2 "" H 650 1150 50  0001 C CNN
+F 3 "" H 650 1150 50  0001 C CNN
+	1    650  1150
 	1    0    0    -1
 $EndComp
@@
 L power:+3.3V #PWR01
 U 1 1 5BE72B85
-P 650 700
-F 0 "#PWR01" H 650 550 50  0001 C CNN
-F 1 "+3.3V" H 665 873 50  0000 C CNN
-F 2 "" H 650 700 50  0001 C CNN
-F 3 "" H 650 700 50  0001 C CNN
-	1    650  700
+P 650 850
+F 0 "#PWR01" H 650 700 50  0001 C CNN
+F 1 "+3.3V" H 665 1023 50  0000 C CNN
+F 2 "" H 650 850 50  0001 C CNN
+F 3 "" H 650 850 50  0001 C CNN
+	1    650  850
 	1    0    0    -1
 $EndComp
