File: kicad/UniBadge-9x9.kicad_pcb (KiCad board)
At the start: 2 copper layers, 50 x 50 mm, 113 parts, among them Q1 2N7002, Q2 2N7002, Q3 2N7002, Q4 2N7002, Q5 2N7002, Q6 2N7002, Q7 2N7002, Q8 2N7002, Q9 2N7002, SW1 SW_DPDT_x2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

Commit message: renamed unibatch to unibadge ... germans...
Routing:
- net VS: track 58.9 -> 62.9 mm, vias 1 -> 2
Other:
- board text added: "UniBadge 9x9"
- board text added: "V1.1"
- board text removed: "UniBatch 9x9"
- board text removed: "V1.0"
Changed lines of the file:
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@@
     (thickness 1.6)
     (drawings 13)
-    (tracks 393)
+    (tracks 396)
     (zones 0)
     (modules 113)
@@
   (module unibatch:smd_switch_slide placed (layer B.Cu)
     (at 6.5 42 270)
-    (fp_text reference SW1 (at 2.5 2.5 90) (layer B.SilkS)
+    (fp_text reference SW1 (at 6.5 0.5 180) (layer B.SilkS)
       (effects (font (size 1 1) (thickness 0.15)) (justify mirror))
     )
@@
     (tags "resistor handsolder")
     (attr smd)
-    (fp_text reference R2 (at 0 1.65) (layer B.SilkS)
+    (fp_text reference R2 (at 0 -1.5) (layer B.SilkS)
       (effects (font (size 1 1) (thickness 0.15)) (justify mirror))
     )
@@
     (tags "resistor handsolder")
     (attr smd)
-    (fp_text reference R1 (at 0 -1.75) (layer B.SilkS)
+    (fp_text reference R1 (at 0 1.5) (layer B.SilkS)
       (effects (font (size 1 1) (thickness 0.15)) (justify mirror))
     )
@@
     (tags "capacitor handsolder")
     (attr smd)
-    (fp_text reference C3 (at 0 1.65) (layer B.SilkS)
+    (fp_text reference C3 (at 0 -1.5) (layer B.SilkS)
       (effects (font (size 1 1) (thickness 0.15)) (justify mirror))
     )
@@
     (tags "capacitor handsolder")
     (attr smd)
-    (fp_text reference C2 (at 0 -1.75 180) (layer B.SilkS)
+    (fp_text reference C2 (at 0 1.5 180) (layer B.SilkS)
       (effects (font (size 1 1) (thickness 0.15)) (justify mirror))
     )
@@
     (tags "capacitor handsolder")
     (attr smd)
-    (fp_text reference C1 (at 0 1.65) (layer B.SilkS)
+    (fp_text reference C1 (at 0 -1.5) (layer B.SilkS)
       (effects (font (size 1 1) (thickness 0.15)) (justify mirror))
     )
@@
     (descr "Through hole straight pin header, 1x02, 2.54mm pitch, single row")
     (tags "Through hole pin header THT 1x02 2.54mm single row")
-    (fp_text reference BT1 (at 0 2.33) (layer B.SilkS)
+    (fp_text reference BT1 (at 0 -5) (layer B.SilkS)
       (effects (font (size 1 1) (thickness 0.15)) (justify mirror))
     )
@@
     (effects (font (size 0.75 0.75) (thickness 0.14)) (justify left mirror))
   )
-  (gr_text V1.0 (at 7.95 15.2) (layer B.SilkS)
+  (gr_text V1.1 (at 7.5 15.2) (layer B.SilkS)
     (effects (font (size 0.5 0.5) (thickness 0.11)) (justify mirror))
   )
-  (gr_text "UniBatch 9x9" (at 23.2 13.208) (layer B.SilkS)
+  (gr_text "UniBadge 9x9" (at 23.2 13.208) (layer B.SilkS)
     (effects (font (size 1.6 1.6) (thickness 0.1875)) (justify left mirror))
   )
@@
   (segment (start 4.5 18) (end 4.5 20.07) (width 0.25) (layer B.Cu) (net 3))
   (segment (start 6.025 37.5) (end 6.025 36) (width 0.25) (layer B.Cu) (net 3))
+  (via (at 4 45) (size 0.8) (drill 0.4) (layers F.Cu B.Cu) (net 3))
+  (segment (start 6.5 42.5) (end 4 45) (width 0.25) (layer B.Cu) (net 3))
+  (segment (start 6.5 42) (end 6.5 42.5) (width 0.25) (layer B.Cu) (net 3))
   (segment (start 6.025 32) (end 6.025 25.405) (width 0.25) (layer B.Cu) (net 4))
   (segment (start 12.525 34) (end 12.525 30.5) (width 0.25) (layer B.Cu) (net 5))

Commit message: fixed clock-enable at cd4017
Parts:
- BT1: value CR2023 -> Battery-Holder (2x AAA)
Connections:
- U2 pad 13: Net-(U2-Pad13) -> GND
Other:
- board text added: "V1.2"
- board text removed: "V1.1"
