File: kicad/UniBadge-9x9.sch (KiCad schematic (older format))
At the start: 108 parts, among them Q1 2N7002, Q2 2N7002, Q3 2N7002, Q4 2N7002, Q5 2N7002, Q6 2N7002, Q7 2N7002, Q8 2N7002, Q9 2N7002, SW1 SW_DPDT_x2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

Commit message: fixed clock-enable at cd4017
Connections:
- net GND: now also U2.13 (CKEN)
- no-connect marks 3 -> 2
Changed lines of the file:
@@
 Wire Wire Line
 	3750 2050 3550 2050
-NoConn ~ 3750 1850
 Connection ~ 10250 3800
 Wire Wire Line
@@
 Wire Wire Line
 	3550 2050 3550 3500
+$Comp
+L power:GND #PWR0101
+U 1 1 5F4025BB
+P 3750 1850
+F 0 "#PWR0101" H 3750 1600 50  0001 C CNN
+F 1 "GND" H 3755 1677 50  0000 C CNN
+F 2 "" H 3750 1850 50  0001 C CNN
+F 3 "" H 3750 1850 50  0001 C CNN
+	1    3750 1850
+	0    1    1    0
+$EndComp
 $EndSCHEMATC
